File: ESP32_MP3_recorder_player_DSP_WIFI_radio/ESP32_MP3_recorder_player_DSP_WIFI_radio.kicad_pcb (KiCad board)
At the start: 2 copper layers, 4 parts, among them J1 Micro_SD_Card_Det, J2 Conn_01x06, U1 ESP32-S3-WROOM-1

Commit message: g
Parts:
- added C1: 100n, Capacitor_SMD:C_0603_1608Metric_Pad1.08x0.95mm_HandSolder, F.Cu at (245.1, -43.2)
- added C10: 100n, Capacitor_SMD:C_0603_1608Metric_Pad1.08x0.95mm_HandSolder, F.Cu at (236.4, -32.9)
- added C11: 15p, Capacitor_SMD:C_0603_1608Metric_Pad1.08x0.95mm_HandSolder, F.Cu at (222.2, -20.1)
- added C12: 10u, Capacitor_SMD:C_0805_2012Metric, F.Cu at (217.8, -23.1)
- added C13: 100n, Capacitor_SMD:C_0603_1608Metric_Pad1.08x0.95mm_HandSolder, F.Cu at (240.7, -40.5)
- added C14: 10u, Capacitor_SMD:C_0805_2012Metric, F.Cu at (232.0, -34.2)
- added C15: 10u, Capacitor_SMD:C_0805_2012Metric, F.Cu at (240.7, -43.2)
- added C16: 100n, Capacitor_SMD:C_0603_1608Metric_Pad1.08x0.95mm_HandSolder, F.Cu at (296.6, -43.3)
- added C17: 10u, Capacitor_SMD:C_0805_2012Metric, F.Cu at (266.6, -34.1)
- added C18: 10u, Capacitor_SMD:C_0805_2012Metric, F.Cu at (271.7, -30.0)
- added C19: 100n, Capacitor_SMD:C_0603_1608Metric_Pad1.08x0.95mm_HandSolder, F.Cu at (296.6, -38.2)
- added C2: 100n, Capacitor_SMD:C_0603_1608Metric_Pad1.08x0.95mm_HandSolder, F.Cu at (245.5, -51.5)
- added C20: 10u, Capacitor_SMD:C_0805_2012Metric, F.Cu at (300.4, -51.5)
- added C21: 10u, Capacitor_SMD:C_0805_2012Metric, F.Cu at (295.9, -51.5)
- added C22: 100n, Capacitor_SMD:C_0603_1608Metric_Pad1.08x0.95mm_HandSolder, F.Cu at (301.0, -41.2)
- added C23: 1u, Capacitor_SMD:C_0603_1608Metric_Pad1.08x0.95mm_HandSolder, F.Cu at (287.8, -36.5)
- added C24: 1u, Capacitor_SMD:C_0603_1608Metric_Pad1.08x0.95mm_HandSolder, F.Cu at (289.2, -31.5)
- added C25: 1u, Capacitor_SMD:C_0603_1608Metric_Pad1.08x0.95mm_HandSolder, F.Cu at (300.3, -46.2)
- added C26: 1u, Capacitor_SMD:C_0603_1608Metric_Pad1.08x0.95mm_HandSolder, F.Cu at (280.4, -27.7)
- added C27: 1u, Capacitor_SMD:C_0603_1608Metric_Pad1.08x0.95mm_HandSolder, F.Cu at (284.8, -27.7)
- added C28: 1u, Capacitor_SMD:C_0603_1608Metric_Pad1.08x0.95mm_HandSolder, F.Cu at (292.3, -39.5)
- added C29: 1u, Capacitor_SMD:C_0603_1608Metric_Pad1.08x0.95mm_HandSolder, F.Cu at (276.1, -30.3)
- added C3: 470n, Capacitor_SMD:C_0805_2012Metric, F.Cu at (226.9, -29.7)
- added C30: 4n7, Capacitor_SMD:C_0603_1608Metric_Pad1.08x0.95mm_HandSolder, F.Cu at (300.3, -48.7)
- added C31: 1u, Capacitor_SMD:C_0603_1608Metric_Pad1.08x0.95mm_HandSolder, F.Cu at (287.8, -39.0)
- added C32: 1u, Capacitor_SMD:C_0603_1608Metric_Pad1.08x0.95mm_HandSolder, F.Cu at (292.3, -42.0)
- added C33: 4n7, Capacitor_SMD:C_0603_1608Metric_Pad1.08x0.95mm_HandSolder, F.Cu at (292.2, -37.0)
- added C34: 10u, Capacitor_SMD:C_0805_2012Metric, F.Cu at (287.9, -41.8)
- added C35: 1u, Capacitor_SMD:C_0603_1608Metric_Pad1.08x0.95mm_HandSolder, F.Cu at (293.6, -34.5)
- added C36: 1u, Capacitor_SMD:C_0603_1608Metric_Pad1.08x0.95mm_HandSolder, F.Cu at (284.8, -30.2)
- added C37: 1u, Capacitor_SMD:C_0603_1608Metric_Pad1.08x0.95mm_HandSolder, F.Cu at (276.1, -27.8)
- added C38: 10u, Capacitor_SMD:C_0805_2012Metric, F.Cu at (196.5, -40.6)
- added C39: 100n, Capacitor_SMD:C_0603_1608Metric_Pad1.08x0.95mm_HandSolder, F.Cu at (200.9, -40.9)
- added C4: 2u2, Capacitor_SMD:C_0805_2012Metric, F.Cu at (245.5, -48.5)
- added C40: 100n, Capacitor_SMD:C_0603_1608Metric_Pad1.08x0.95mm_HandSolder, F.Cu at (205.2, -39.8)
- added C5: DNP, Capacitor_SMD:C_0603_1608Metric_Pad1.08x0.95mm_HandSolder, F.Cu at (231.2, -26.9)
- added C6: 100n, Capacitor_SMD:C_0603_1608Metric_Pad1.08x0.95mm_HandSolder, F.Cu at (235.6, -30.4)
- added C7: 100n, Capacitor_SMD:C_0603_1608Metric_Pad1.08x0.95mm_HandSolder, F.Cu at (236.4, -35.4)
- added C8: 10u, Capacitor_SMD:C_0805_2012Metric, F.Cu at (222.4, -25.8)
- added C9: 10u, Capacitor_SMD:C_0805_2012Metric, F.Cu at (217.8, -20.1)
- added D1: LED_Small, LED_SMD:LED_0805_2012Metric, F.Cu at (235.7, -38.2)
- added D2: LED_Small, LED_SMD:LED_0805_2012Metric, F.Cu at (220.6, -52.3)
- added J10: AudioJack4_SwitchTR1, Z_mycustom_footprint_lib:PJ-316A-6A, F.Cu at (195.1, -48.0)
- added J3: Conn_01x06, Connector_PinHeader_2.54mm:PinHeader_1x06_P2.54mm_Vertical, F.Cu at (116.6, 63.8)
- added J4: AUDIO, Connector_PinHeader_2.54mm:PinHeader_1x03_P2.54mm_Vertical, F.Cu at (276.0, -38.9)
- added J5: AUDIO, Connector_PinHeader_2.54mm:PinHeader_1x03_P2.54mm_Vertical, F.Cu at (271.4, -38.9)
- added J6: AUDIO, Connector_PinHeader_2.54mm:PinHeader_1x03_P2.54mm_Vertical, F.Cu at (291.4, -50.7)
- added J7: AudioJack4_SwitchTR1, Z_mycustom_footprint_lib:PJ-316A-6A, F.Cu at (62.1, 91.7)
- added J8: AUDIO, Connector_PinHeader_2.54mm:PinHeader_1x03_P2.54mm_Vertical, F.Cu at (286.7, -50.7)
- added J9: Conn_01x06, Connector_PinHeader_2.54mm:PinHeader_1x06_P2.54mm_Vertical, F.Cu at (120.8, 63.8)
- added L1: L_Small, Inductor_SMD:L_0603_1608Metric, F.Cu at (217.9, -26.0)
- added R10: 1Meg, Resistor_SMD:R_0603_1608Metric_Pad0.98x0.95mm_HandSolder, F.Cu at (249.9, -48.8)
- added R11: 10, Resistor_SMD:R_0402_1005Metric, F.Cu at (254.3, -51.7)
- added R12: 10, Resistor_SMD:R_0402_1005Metric, F.Cu at (231.3, -30.0)
- added R13: 10, Resistor_SMD:R_0402_1005Metric, F.Cu at (240.1, -38.0)
- added R14: 10, Resistor_SMD:R_0402_1005Metric, F.Cu at (245.4, -45.7)
- added R15: 10, Resistor_SMD:R_0402_1005Metric, F.Cu at (254.3, -49.2)
- added R16: 10, Resistor_SMD:R_0402_1005Metric, F.Cu at (249.9, -46.3)
- added R17: 10k, Resistor_SMD:R_0603_1608Metric_Pad0.98x0.95mm_HandSolder, F.Cu at (258.7, -51.7)
- added R18: 10k, Resistor_SMD:R_0603_1608Metric_Pad0.98x0.95mm_HandSolder, F.Cu at (225.9, -19.2)
- added R19: 10k, Resistor_SMD:R_0603_1608Metric_Pad0.98x0.95mm_HandSolder, F.Cu at (244.3, -38.4)
- added R2: 1k, Resistor_SMD:R_0603_1608Metric_Pad0.98x0.95mm_HandSolder, F.Cu at (222.3, -22.9)
- added R20: 10k, Resistor_SMD:R_0603_1608Metric_Pad0.98x0.95mm_HandSolder, F.Cu at (239.2, -30.6)
- added R21: 10k, Resistor_SMD:R_0603_1608Metric_Pad0.98x0.95mm_HandSolder, F.Cu at (253.5, -47.0)
- added R22: 10k, Resistor_SMD:R_0603_1608Metric_Pad0.98x0.95mm_HandSolder, F.Cu at (206.5, -16.0)
- added R23: 10k, Resistor_SMD:R_0603_1608Metric_Pad0.98x0.95mm_HandSolder, F.Cu at (240.1, -33.2)
- added R24: 10, Resistor_SMD:R_0402_1005Metric, F.Cu at (234.9, -27.7)
- added R25: 10, Resistor_SMD:R_0402_1005Metric, F.Cu at (212.3, -16.0)
- added R26: 27, Resistor_SMD:R_0402_1005Metric, F.Cu at (209.4, -16.0)
- added R27: 10, Resistor_SMD:R_0402_1005Metric, F.Cu at (230.5, -24.7)
- added R28: 10, Resistor_SMD:R_0402_1005Metric, F.Cu at (289.2, -34.0)
- added R29: 10, Resistor_SMD:R_0402_1005Metric, F.Cu at (295.9, -45.8)
- added R3: 1k, Resistor_SMD:R_0603_1608Metric_Pad0.98x0.95mm_HandSolder, F.Cu at (226.8, -26.7)
- added R30: 27, Resistor_SMD:R_0402_1005Metric, F.Cu at (284.9, -32.7)
- added R31: 10, Resistor_SMD:R_0402_1005Metric, F.Cu at (280.5, -32.7)
- added R32: 27, Resistor_SMD:R_0402_1005Metric, F.Cu at (280.4, -30.2)
- added R33: 27, Resistor_SMD:R_0402_1005Metric, F.Cu at (296.6, -40.8)
- added R34: 27, Resistor_SMD:R_0402_1005Metric, F.Cu at (301.0, -43.7)
- added R35: 1k, Resistor_SMD:R_0603_1608Metric_Pad0.98x0.95mm_HandSolder, F.Cu at (289.1, -29.0)
- added R36: 2k7, Resistor_SMD:R_0603_1608Metric_Pad0.98x0.95mm_HandSolder, F.Cu at (293.6, -32.0)
- added R37: 2k7, Resistor_SMD:R_0603_1608Metric_Pad0.98x0.95mm_HandSolder, F.Cu at (295.9, -48.5)
- added R38: 1k, Resistor_SMD:R_0603_1608Metric_Pad0.98x0.95mm_HandSolder, F.Cu at (249.5, -16.6)
- added R39: 1k, Resistor_SMD:R_0603_1608Metric_Pad0.98x0.95mm_HandSolder, F.Cu at (249.5, -19.1)
- added R4: 300, Resistor_SMD:R_0603_1608Metric_Pad0.98x0.95mm_HandSolder, F.Cu at (249.9, -51.5)
- added R40: 1k, Resistor_SMD:R_0603_1608Metric_Pad0.98x0.95mm_HandSolder, F.Cu at (249.4, -13.2)
- added R41: 1k, Resistor_SMD:R_0603_1608Metric_Pad0.98x0.95mm_HandSolder, F.Cu at (253.8, -16.6)
- added R42: 1k, Resistor_SMD:R_0603_1608Metric_Pad0.98x0.95mm_HandSolder, F.Cu at (245.1, -13.2)
- added R43: 1k, Resistor_SMD:R_0603_1608Metric_Pad0.98x0.95mm_HandSolder, F.Cu at (253.8, -19.1)
- added R44: 100k, Resistor_SMD:R_0805_2012Metric, F.Cu at (245.1, -15.9)
- added R45: 100k, Resistor_SMD:R_0805_2012Metric, F.Cu at (245.1, -18.9)
- added R5: 300, Resistor_SMD:R_0603_1608Metric_Pad0.98x0.95mm_HandSolder, F.Cu at (222.2, -17.6)
- added R6: 10k, Resistor_SMD:R_0603_1608Metric_Pad0.98x0.95mm_HandSolder, F.Cu at (226.7, -21.5)
- added R7: 5k1, Resistor_SMD:R_0603_1608Metric_Pad0.98x0.95mm_HandSolder, F.Cu at (245.1, -40.7)
- added R8: 5k1, Resistor_SMD:R_0603_1608Metric_Pad0.98x0.95mm_HandSolder, F.Cu at (217.8, -17.3)
- added R9: 10k, Resistor_SMD:R_0603_1608Metric_Pad0.98x0.95mm_HandSolder, F.Cu at (240.8, -35.5)
- added SW1: MCU_RESET, SamacSys_Parts:PTS526SK15SMTR2LFS, F.Cu at (219.6, -31.5)
- added SW2: MCU_RESET, SamacSys_Parts:PTS526SK15SMTR2LFS, F.Cu at (210.6, -21.1)
- added TP1: TestPoint_THT, TestPoint:TestPoint_Loop_D2.60mm_Drill0.9mm_Beaded, F.Cu at (235.9, -42.2)
- added TP2: TestPoint_THT, TestPoint:TestPoint_Loop_D2.60mm_Drill0.9mm_Beaded, F.Cu at (249.4, -43.2)
- added TP3: TestPoint_THT, TestPoint:TestPoint_Loop_D2.60mm_Drill0.9mm_Beaded, F.Cu at (266.9, -29.0)
- added U2: ESP32-S3-WROOM-1, Espressif:ESP32-S3-WROOM-1, F.Cu at (78.9, 66.4)
- added U3: AMS1117-3.3, Package_TO_SOT_SMD:SOT-223-3_TabPin2, F.Cu at (238.3, -48.9)
- added U4: TLV320AIC3254, Package_DFN_QFN:QFN-32-1EP_5x5mm_P0.5mm_EP3.1x3.1mm_ThermalVias, F.Cu at (83.0, 88.7)
- added U5: TPA2012D2, Package_DFN_QFN:QFN-20-1EP_4x4mm_P0.5mm_EP2.6x2.6mm_ThermalVias, F.Cu at (212.8, -44.1)
- added U6: PCA9557PW, Package_SO:TSSOP-16_4.4x5mm_P0.65mm, F.Cu at (214.0, -50.6)
- J1: value Micro_SD_Card_Det -> USB_C_Receptacle; footprint Connector_Card:microSD_HC_Molex_104031-0811 -> Connector_USB:USB_C_Receptacle_HRO_TYPE-C-31-M-12
- J2: value Conn_01x06 -> Micro_SD_Card_Det; footprint Connector_PinHeader_2.54mm:PinHeader_1x06_P2.54mm_Vertical -> Connector_Card:microSD_HC_Molex_104031-0811
- R1: value 10k -> 2k7
- U1: value ESP32-S3-WROOM-1 -> SRV05-4; footprint Espressif:ESP32-S3-WROOM-1 -> Package_TO_SOT_SMD:SOT-23-6
- moved J1 214.4 mm to (53.4, 75.1), turned to -90 degrees
- moved U1 183.3 mm to (61.4, 75.0)
- moved J2 153.0 mm to (105.5, 63.3)
- moved R1 81.3 mm to (226.8, -24.0)
Connections:
- J2 pad 1: GND -> /DATA_2
- J2 pad 2: +3V3 -> /DATA_3
- J2 pad 3: GND -> /CMD
- J2 pad 4: /I2S_1_SCK -> +3V3
- J2 pad 5: /I2S_1_SD -> /CLK
- J2 pad 6: /I2S_1_WS -> GND
- R1 pad 1: /CARD_DETECT -> +5V
- R1 pad 2: +3V3 -> Net-(R1-Pad2)
- U1 pad 1: GND -> unconnected-(U1-Pad1)
- U1 pad 2: +3V3 -> GND
- U1 pad 3: /ESP_EN -> unconnected-(U1-Pad3)
- U1 pad 4: GPIO_4 -> D+
- U1 pad 5: GPIO_5 -> VBUS
- U1 pad 6: GPIO_6 -> D-
Other:
- board outline added: 100 x 100 mm
