File: ESP32_MP3_recorder_player_DSP_WIFI_radio/ESP32_MP3_recorder_player_DSP_WIFI_radio.kicad_sch (KiCad schematic)
At the start: 38 parts, among them J1 Micro_SD_Card_Det, J2 Conn_01x06, U1 ESP32-S3-WROOM-1

Commit message: 5
Parts:
- added U?: TLV320AIC3254, Package_DFN_QFN:QFN-32-1EP_5x5mm_P0.5mm_EP3.1x3.1mm_ThermalVias, symbol My_custom_lib:TLV320AIC3254
Connections:
- net GND: now also U?.17 (AVSS), U?.28 (DVSS), U?.33 (EP), U?.7 (IOVSS)
Changed lines of the file:
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@@
+    (stroke (width 0) (type default) (color 0 0 0 0))
+  )
+  (wire (pts (xy 87.63 243.84) (xy 87.63 246.38))
     (stroke (width 0) (type default) (color 0 0 0 0))
   )
@@
     (stroke (width 0) (type default) (color 0 0 0 0))
   )
+  (wire (pts (xy 90.17 243.84) (xy 90.17 246.38))
+    (stroke (width 0) (type default) (color 0 0 0 0))
+  )
   (wire (pts (xy 237.49 33.02) (xy 248.92 33.02))
     (stroke (width 0) (type default) (color 0 0 0 0))
@@
     (stroke (width 0) (type default) (color 0 0 0 0))
   )
+  (wire (pts (xy 92.71 243.84) (xy 92.71 246.38))
+    (stroke (width 0) (type default) (color 0 0 0 0))
+  )
   (wire (pts (xy 233.68 207.01) (xy 233.68 209.55))
     (stroke (width 0) (type default) (color 0 0 0 0))
@@
   )
   (wire (pts (xy 254 210.82) (xy 254 207.01))
+    (stroke (width 0) (type default) (color 0 0 0 0))
+  )
+  (wire (pts (xy 85.09 243.84) (xy 85.09 246.38))
     (stroke (width 0) (type default) (color 0 0 0 0))
   )
@@
     )
     (property "Datasheet" "" (id 3) (at 270.51 259.08 0)
+      (effects (font (size 1.27 1.27)) hide)
+    )
+    (pin "1")
+  )
+  (symbol (lib_id "power:GND") (at 85.09 246.38 0) (unit 1)
+    (in_bom yes) (on_board yes) (fields_autoplaced)
+    (property "Reference" "#PWR?" (id 0) (at 85.09 252.73 0)
+      (effects (font (size 1.27 1.27)) hide)
+    )
+    (property "Value" "GND" (id 1) (at 85.09 251.46 0)
+      (effects (font (size 1.27 1.27)) hide)
+    )
+    (property "Footprint" "" (id 2) (at 85.09 246.38 0)
+      (effects (font (size 1.27 1.27)) hide)
+    )
+    (property "Datasheet" "" (id 3) (at 85.09 246.38 0)
       (effects (font (size 1.27 1.27)) hide)
     )
@@
     (pin "2")
   )
+  (symbol (lib_id "power:GND") (at 90.17 246.38 0) (unit 1)
+    (in_bom yes) (on_board yes) (fields_autoplaced)
+    (property "Reference" "#PWR?" (id 0) (at 90.17 252.73 0)
+      (effects (font (size 1.27 1.27)) hide)
+    )
+    (property "Value" "GND" (id 1) (at 90.17 251.46 0)
+      (effects (font (size 1.27 1.27)) hide)
+    )
+    (property "Footprint" "" (id 2) (at 90.17 246.38 0)
+      (effects (font (size 1.27 1.27)) hide)
+    )
+    (property "Datasheet" "" (id 3) (at 90.17 246.38 0)
+      (effects (font (size 1.27 1.27)) hide)
+    )
+    (pin "1")
+  )
   (symbol (lib_id "power:GND") (at 116.84 -31.75 0) (mirror y) (unit 1)
     (in_bom yes) (on_board yes) (fields_autoplaced)
@@
     (pin "2")
   )
+  (symbol (lib_id "power:GND") (at 92.71 246.38 0) (unit 1)
+    (in_bom yes) (on_board yes) (fields_autoplaced)
+    (property "Reference" "#PWR?" (id 0) (at 92.71 252.73 0)
+      (effects (font (size 1.27 1.27)) hide)
+    )
+    (property "Value" "GND" (id 1) (at 92.71 251.46 0)
+      (effects (font (size 1.27 1.27)) hide)
+    )
+    (property "Footprint" "" (id 2) (at 92.71 246.38 0)
+      (effects (font (size 1.27 1.27)) hide)
+    )
+    (property "Datasheet" "" (id 3) (at 92.71 246.38 0)
+      (effects (font (size 1.27 1.27)) hide)
+    )
+    (pin "1")
+  )
   (symbol (lib_id "power:VBUS") (at 321.31 36.83 0) (mirror y) (unit 1)
     (in_bom yes) (on_board yes) (fields_autoplaced)
@@
     (pin "1")
   )
+  (symbol (lib_id "power:GND") (at 87.63 246.38 0) (unit 1)
+    (in_bom yes) (on_board yes) (fields_autoplaced)
+    (property "Reference" "#PWR?" (id 0) (at 87.63 252.73 0)
+      (effects (font (size 1.27 1.27)) hide)
+    )
+    (property "Value" "GND" (id 1) (at 87.63 251.46 0)
+      (effects (font (size 1.27 1.27)) hide)
+    )
+    (property "Footprint" "" (id 2) (at 87.63 246.38 0)
+      (effects (font (size 1.27 1.27)) hide)
+    )
+    (property "Datasheet" "" (id 3) (at 87.63 246.38 0)
+      (effects (font (size 1.27 1.27)) hide)
+    )
+    (pin "1")
+  )
   (symbol (lib_id "Device:LED_Small") (at 116.84 -46.99 90) (unit 1)
     (in_bom yes) (on_board yes) (fields_autoplaced)
@@
     (pin "1")
     (pin "2")
+  )
+  (symbol (lib_id "My_custom_lib:TLV320AIC3254") (at 87.63 208.28 0) (unit 1)
+    (in_bom yes) (on_board yes) (fields_autoplaced)
+    (property "Reference" "U?" (id 0) (at 94.7294 243.84 0)
+      (effects (font (size 1.27 1.27)) (justify left))
+    )
+    (property "Value" "TLV320AIC3254" (id 1) (at 94.7294 246.38 0)
+      (effects (font (size 1.27 1.27)) (justify left))
+    )
+    (property "Footprint" "Package_DFN_QFN:QFN-32-1EP_5x5mm_P0.5mm_EP3.1x3.1mm_ThermalVias" (id 2) (at 81.28 168.91 0)
+      (effects (font (size 1.27 1.27)) hide)
+    )
+    (property "Datasheet" "https://www.ti.com/cn/lit/ds/symlink/tlv320aic3254.pdf?ts=1676901627751&ref_url=https%253A%252F%252Fjlcpcb.com%252F" (id 3) (at 81.28 163.83 0)
+      (effects (font (size 1.27 1.27)) hide)
+    )
+    (property "SITE" "https://jlcpcb.com/partdetail/TexasInstruments-TLV320AIC3254IRHBR/C9925" (id 4) (at 82.55 166.37 0)
+      (effects (font (size 1.27 1.27)) hide)
+    )
+    (property "LCSC" "C9925" (id 5) (at 88.9 161.29 0)
+      (effects (font (size 1.27 1.27)) hide)
+    )
+    (pin "1")
+    (pin "10")
+    (pin "11")
+    (pin "12")
+    (pin "13")
+    (pin "14")
+    (pin "15")
+    (pin "16")
+    (pin "17")
+    (pin "18")
+    (pin "19")
+    (pin "2")
+    (pin "20")
+    (pin "21")
+    (pin "22")
+    (pin "23")
+    (pin "24")
+    (pin "25")
+    (pin "26")
+    (pin "27")
+    (pin "28")
+    (pin "29")
+    (pin "3")
+    (pin "30")
+    (pin "31")
+    (pin "32")
+    (pin "33")
+    (pin "4")
+    (pin "5")
+    (pin "6")
+    (pin "7")
+    (pin "8")
+    (pin "9")
   )
   (symbol (lib_id "power:+3V3") (at 25.4 100.33 0) (unit 1)
@@
       (reference "#PWR0101") (unit 1) (value "GND") (footprint "")
     )
+    (path "/09f27143-e440-4cf6-8bae-f492d2acc983"
+      (reference "#PWR?") (unit 1) (value "GND") (footprint "")
+    )
     (path "/13304213-8343-4faf-856a-98a7288d0e1e"
       (reference "#PWR?") (unit 1) (value "+3V3") (footprint "")
@@
       (reference "#PWR?") (unit 1) (value "GND") (footprint "")
     )
+    (path "/5e5e9384-2ccd-4f0f-bc88-1e158a14b27b"
+      (reference "#PWR?") (unit 1) (value "GND") (footprint "")
+    )
     (path "/64a36764-e37f-457c-88e2-e8e1a16d55fc"
       (reference "#PWR?") (unit 1) (value "GND") (footprint "")
@@
       (reference "#PWR?") (unit 1) (value "GND") (footprint "")
     )
+    (path "/79104528-79b9-4f19-9dca-03c824441315"
+      (reference "#PWR?") (unit 1) (value "GND") (footprint "")
+    )
     (path "/8381c349-c0a2-4e3b-aa4e-38f1264f3c3a"
       (reference "#PWR?") (unit 1) (value "VBUS") (footprint "")
@@
       (reference "#PWR?") (unit 1) (value "GND") (footprint "")
     )
+    (path "/be0693c7-6f3a-4087-b868-90f2bc5e7cf2"
+      (reference "#PWR?") (unit 1) (value "GND") (footprint "")
+    )
     (path "/c00cbabd-4487-498c-9030-17e1a16f5632"
       (reference "#PWR?") (unit 1) (value "GND") (footprint "")
@@
       (reference "U?") (unit 1) (value "AMS1117-3.3") (footprint "Package_TO_SOT_SMD:SOT-223-3_TabPin2")
     )
+    (path "/e69217d3-4112-43ec-8b50-d5835a83f0dc"
+      (reference "U?") (unit 1) (value "TLV320AIC3254") (footprint "Package_DFN_QFN:QFN-32-1EP_5x5mm_P0.5mm_EP3.1x3.1mm_ThermalVias")
+    )
     (path "/f80d167b-1df0-4a46-89bf-850110c2d398"

Commit message: g
Parts:
- removed C?: 10u, Capacitor_SMD:C_0805_2012Metric, symbol Device:C_Small
- removed C?: 15n, Capacitor_SMD:C_0603_1608Metric_Pad1.08x0.95mm_HandSolder, symbol Device:C_Small
- removed C?: 2u2, Capacitor_SMD:C_0805_2012Metric, symbol Device:C
- removed C?: 470n, Capacitor_SMD:C_0805_2012Metric, symbol Device:C
- removed D?: D_Small, Diode_SMD:D_SOD-123, symbol Device:D_Small
- removed D?: LED_Small, LED_SMD:LED_0805_2012Metric, symbol Device:LED_Small
- removed J?: Conn_01x02, Connector_PinHeader_2.54mm:PinHeader_1x02_P2.54mm_Vertical, symbol Connector_Generic:Conn_01x02
- removed L?: L_Small, Inductor_SMD:L_0805_2012Metric, symbol Device:L_Small
- removed R?: 150k, Resistor_SMD:R_0805_2012Metric, symbol Device:R
- removed R?: 100k, Resistor_SMD:R_0805_2012Metric, symbol Device:R
- removed R?: 300, Resistor_SMD:R_0603_1608Metric_Pad0.98x0.95mm_HandSolder, symbol Device:R_Small
- removed R?: 1Meg, Resistor_SMD:R_0603_1608Metric_Pad0.98x0.95mm_HandSolder, symbol Device:R_Small
- removed R?: 2k2, Resistor_SMD:R_0805_2012Metric, symbol Device:R
- removed U?: TLV320AIC3254, Package_DFN_QFN:QFN-32-1EP_5x5mm_P0.5mm_EP3.1x3.1mm_ThermalVias, symbol My_custom_lib:TLV320AIC3254
- added FB1: FerriteBead_Small, symbol Device:FerriteBead_Small
- added R10, R11, R19, R20, R22, R23, R24, R26, R6, R7, R8, R9: 10, Resistor_SMD:R_0402_1005Metric, symbol Device:R_Small
- added R13, R14, R15, R16, R17, R18: 10k, Resistor_SMD:R_0603_1608Metric_Pad0.98x0.95mm_HandSolder, symbol Device:R_Small
- added R21, R25, R27, R28, R29: 27, Resistor_SMD:R_0402_1005Metric, symbol Device:R_Small
- gave numbers to parts that had none: 21
- renumbered J1 to J2, J2 to J3, R1 to R12, U1 to U2
Connections:
- net +3V3: now also R13.2, R14.2, R15.2, R16.2, R17.2, R18.2
- net +5V: now also FB1.1
- net CARD_DETECT: now also R18.1, R19.1; no longer R12.1
- net CLK: now also R11.1, R17.1
- net CMD: now also R10.1, R16.1
- net DATA_0: now also R12.1, R6.1
- net DATA_1: now also R13.1, R7.1
- net DATA_2: now also R14.1, R8.1
- net DATA_3: now also R15.1, R9.1
- net GND: no longer J3.3 (Pin_3)
- net GPIO_1: now also R8.2
- net GPIO_11: now also R28.1
- net GPIO_12: now also R29.1
- net GPIO_14: now also R25.1
- net GPIO_2: now also R9.2
- net GPIO_21: now also R27.1
- net GPIO_36: now also R20.1
- net GPIO_37: now also R22.1
- net GPIO_38: now also R24.1
- net GPIO_39: now also R26.1
- net GPIO_40: now also R19.2
- net GPIO_41: now also R7.2
- net GPIO_42: now also R6.2
- net GPIO_43: now also R10.2
- net GPIO_44: now also R11.2
- net GPIO_47: now also R23.1
- net GPIO_48: now also R21.1
- net I2S_1_SCK: now also R24.2
- net I2S_1_SD: now also R22.2
- net I2S_1_WS: now also R20.2
- net VBUS: now also FB1.2
- new net Audio_Codec/BCLK: R27.2
- new net Audio_Codec/DIN: R29.2
- new net Audio_Codec/DOUT: R28.2
- new net Audio_Codec/MCLK: R23.2
- new net Audio_Codec/RESET: R21.2
- new net Audio_Codec/WCLK: R25.2
- new net I2S_1_X: J3.3 (Pin_3), R26.2
- no-connect marks 10 -> 13
Other:
- added sheet Audio_Codec (Audio_Codec.kicad_sch)
- moved on the sheet: C8, C9, J2, J3, R12
