File: ESP32_MP3_recorder_player_DSP_WIFI_radio/ESP32_MP3_recorder_player_DSP_WIFI_radio.kicad_sch (KiCad schematic)
At the start: 49 parts, among them J1 USB_C_Receptacle, J2 Micro_SD_Card_Det, J3 Conn_01x06, SW1 MCU_RESET, SW2 MCU_RESET, U1 SRV05-4, U2 ESP32-S3-WROOM-1, U3 AMS1117-3.3

Commit message: d
Parts:
- removed R12, R13, R14, R15, R16, R17, R18: 10k, Resistor_SMD:R_0603_1608Metric_Pad0.98x0.95mm_HandSolder, symbol Device:R_Small
- added BT?: Battery_Cell, Connector_PinHeader_2.54mm:PinHeader_1x02_P2.54mm_Vertical, symbol Device:Battery_Cell
- added C? (x9): 10u, Capacitor_SMD:C_0805_2012Metric, symbol Device:C_Small
- added C?: 100n, Capacitor_SMD:C_0603_1608Metric_Pad1.08x0.95mm_HandSolder, symbol Device:C_Small
- added D? (x2): D_Schottky, Diode_SMD:D_SMA_Handsoldering, symbol Device:D_Schottky
- added D? (x2): green, LED_SMD:LED_0805_2012Metric, symbol Device:LED_Small
- added J?: Conn_01x03, Connector_PinHeader_2.54mm:PinHeader_1x03_P2.54mm_Vertical, symbol Connector_Generic:Conn_01x03
- added J?: Conn_01x02, Connector_PinHeader_2.54mm:PinHeader_1x02_P2.54mm_Vertical, symbol Connector_Generic:Conn_01x02
- added L?: L_Small, Inductor_SMD:L_0603_1608Metric, symbol Device:L_Small
- added L?: L_Small, symbol Device:L_Small
- added Q?: nMOS, Package_TO_SOT_SMD:SOT-23, symbol Device:Q_NMOS_GSD
- added R? (x7): 10k, Resistor_SMD:R_0402_1005Metric, symbol Device:R_Small
- added R?: 10k, Resistor_SMD:R_0603_1608Metric_Pad0.98x0.95mm_HandSolder, symbol Device:R_Small
- added R?: 1k, Resistor_SMD:R_0805_2012Metric, symbol Device:R
- added R?: 0R2, Resistor_SMD:R_0603_1608Metric_Pad0.98x0.95mm_HandSolder, symbol Device:R_Small
- added U?: TP5000, Package_DFN_QFN:QFN-16-1EP_4x4mm_P0.65mm_EP2.5x2.5mm_ThermalVias, symbol My_custom_lib:TP5000
- added U?: AMS1117-3.3, Package_TO_SOT_SMD:SOT-223-3_TabPin2, symbol Regulator_Linear:AMS1117-3.3
Connections:
- net +3V3: now also C?.1, C?.1, D?.2 (A), L?.2, R?.2, R?.2, R?.2, R?.2, R?.2, R?.2, R?.2, U?.2 (VO)
- net +5V: now also C?.1, C?.1, D?.1 (K), J?.3 (Pin_3), R?.1, U?.1 (VIN), U?.16 (VIN), U?.2 (VIN), U?.3 (VI)
- net CARD_DETECT: now also R?.1
- net CLK: now also R?.1
- net CMD: now also R?.1
- net DATA_0: now also R?.1
- net DATA_1: now also R?.1
- net DATA_2: now also R?.1
- net DATA_3: now also R?.1
- net GND: now also BT?.2 (-), C?.2, C?.2, C?.2, C?.2, C?.2, C?.2, C?.2, C?.2, C?.2, C?.2, D?.2 (A), J?.1 (Pin_1), Q?.2 (S), R?.1, U?.1 (GND), U?.12 (RTRICK), U?.6 (GND), U?.7 (GND)
- new net: D?.1 (K), L?.1, U?.3 (LX), U?.4 (LX), U?.5 (LX)
- new net: J?.2 (Pin_2), Q?.1 (G), R?.2
- new net: BT?.1 (+), C?.1, C?.1, C?.1, L?.1, R?.1, U?.9 (BAT)
- new net: J?.2 (Pin_2), U?.11 (TS)
- new net: C?.1, U?.10 (VREG)
- new net: D?.1 (K), U?.14 (~{CHRG})
- new net: D?.1 (K), U?.15 (~{STDBY})
- new net: C?.1, C?.1, L?.2, R?.2, U?.8 (VS)
- new net: D?.2 (A), D?.2 (A), R?.2
- new net CS: Q?.3 (D), U?.13 (CS)
- no-connect marks 13 -> 16
Other:
- note added: "500mA @3.6V 1.8W => 400mA @5V 2W"
- note added: "RShunt (Ω) IBAT (mA) 1 100 0.2 500 0.1 1000 0.067 1500 0.05 2000"
