File: ESP32_MP3_recorder_player_DSP_WIFI_radio/Audio_Codec.kicad_sch (KiCad schematic)
At the start: 59 parts, among them J4 AUDIO, J5 AUDIO, J6 AUDIO, J7 AudioJack4_SwitchTR1, J8 AudioJack4_SwitchTR1, J9 Conn_01x06, U4 TLV320AIC3254, U5 TPA2012D2, U6 PCA9557PW

Commit message: d
Parts:
- removed C35: 100n, Capacitor_SMD:C_0603_1608Metric_Pad1.08x0.95mm_HandSolder, symbol Device:C_Small
- removed D1, D2: LED_Small, LED_SMD:LED_0805_2012Metric, symbol Device:LED_Small
- removed J4: AUDIO, Connector_PinHeader_2.54mm:PinHeader_1x03_P2.54mm_Vertical, symbol Connector_Generic:Conn_01x03
- removed J7: AudioJack4_SwitchTR1, Z_mycustom_footprint_lib:PJ-316A-6A, symbol Connector:AudioJack4_SwitchTR1
- removed R40: 2k7, Resistor_SMD:R_0603_1608Metric_Pad0.98x0.95mm_HandSolder, symbol Device:R_Small
- removed R41, R42: 1k, Resistor_SMD:R_0603_1608Metric_Pad0.98x0.95mm_HandSolder, symbol Device:R_Small
- removed R43, R46: 300, Resistor_SMD:R_0603_1608Metric_Pad0.98x0.95mm_HandSolder, symbol Device:R_Small
- removed TP2, TP3: TestPoint_THT, TestPoint:TestPoint_Loop_D2.60mm_Drill0.9mm_Beaded, symbol Connector:TestPoint
- removed U6: PCA9557PW, Package_SO:TSSOP-16_4.4x5mm_P0.65mm, symbol Interface_Expansion:PCA9557PW
Connections:
- net GND: no longer U5.17 (OUTR-), U5.5 (OUTL-)
- net GPIO_6: now reaches U5.15 (G0)
- net GPIO_4: now reaches U5.8 (~{SDR})
- net GPIO_4: now also U5.7 (~{SDL})
- net GPIO_5: now reaches U5.1 (G1)
- net at C29.2: now also U5.20 (INL+); no longer U5.19 (INL-)
- net at U5.17 (OUTR-): now also C30.2; no longer C34.2
- net at C26.2: now also U5.19 (INL-); no longer U5.20 (INL+)
- new net: C34.2, U5.18 (INR+)
- no-connect marks 3 -> 0
Other:
- note removed: "0011[A2][A1][A0]"
- moved on the sheet: C20, C21, C22, C23, C26, C28, C29, C30, C32, C34, L1, U5
